File: buck-tpsm33610.kicad_pcb (KiCad board)
At the start: 2 copper layers, 9 x 12.5 mm, 17 parts, among them J1 1x03, U1 TPSM33610S3Q

Commit message: buck-tpsm33610: rotate C1, swap R4/C2, and fix the resistance measurement basis
C1 turns 180 so its VIN pad faces U1 instead of away from it. The VIN run now
stops at the east pad, 2.95 mm short of where it used to, and never crosses
under the body; the C1 -> J1.1 leg climbs the east side; C1's GND stub and its
via move to the west pad. C2 and R4 swap so the input cap, not a 0R EN pull-up
carrying ~10 nA, sits hard against U1's pin row (SNVSCS7E 8.5.1 item 1).

The 0.72 mm VIN vertical starts at y 5.050, not 4.889: at that width the round
end cap reaches 0.36 mm below the start point and /EN's top edge is at 4.485,
which left 0.044 mm against a 0.15 mm rule. 5.050 puts the cap 0.205 mm clear
and the endpoint still lands inside the 0.44 mm horizontal.

MEASUREMENT BASIS, and the reason every earlier number in this file was wrong:
copper_guards resistance at its default --grid 0.2 under-resolves this board.
The GND solve comes out EXACTLY SINGULAR -- nan mOhm, guard exits 2 -- and that
is pre-existing, not caused by the rotation: the un-rotated board is equally
singular at 0.2. At --grid 0.1 both GND paths solve. The same coarse grid also
inflated /VIN C1.1<->U1.3 to 12.259 mOhm. All six paths below are --grid 0.1,
--oz 2, both ends measured the same way:

  path                  rot 0    rot 180   budget
  /VIN  C1.1 <-> U1.3   6.134    4.642     5   (budget is un-derived; see below)
  /VIN  J1.1 <-> U1.3   7.372    5.525     25
  GND   J1.2 <-> U1.10  1.427    1.818     10
  GND   C2.2 <-> U1.10  1.332    1.333     5
  /VOUT J1.3 <-> U1.4     --     0.918     10
  /VOUT U1.4 <-> C4.1     --     0.479     3

So the rotation buys 1.49 mOhm on the bulk path and 1.85 from the header, and
pays 0.39 on GND -- a fifth of the 3.38 mOhm claimed off the coarse grid.

The 5 mOhm on /VIN C1.1<->U1.3 and the 3 nH CIN_HF figure in the plan were both
set by me during planning with no failure mode behind them, and neither ever
entered this repo as a constraint. Treat them as target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
Parts:
- moved R4 1.66 mm to (101.3, 100.4)
- moved C2 0.93 mm to (101.2, 99.1)
- turned C1 to 180 degrees
Routing:
- net /VIN: track 13.9 -> 10.2 mm
- net /EN: track 8.11 -> 10.9 mm
